Commit message: Issues solved & navigation done

File: articubot_one/description/lidar.xacro (robot description, xacro)
@@ -4,5 +4,5 @@
         <parent link="base_link"/>
         <child link="laser_frame"/>
-        <origin xyz="-0.065 0 0.191" rpy="0 0 0"/>
+        <origin xyz="-0.055 0 0.141" rpy="0 0 3.1416"/>
     </joint>
     <link name="laser_frame">

File: articubot_one/description/robot_core.xacro (robot description, xacro)
@@ -73,5 +73,5 @@
         <parent link="base_link"/>
         <child link="left_wheel"/>
-        <origin xyz="0 ${wheel_offset_y} ${wheel_radius}" rpy="-${pi/2} 0 0" />
+        <origin xyz="-0.01 ${wheel_offset_y} ${wheel_radius}" rpy="-${pi/2} 0 0" />
         <axis xyz="0 0 1"/>
     </joint>
@@ -99,5 +99,5 @@
         <parent link="base_link"/>
         <child link="right_wheel"/>
-        <origin xyz="0 ${-wheel_offset_y} ${wheel_radius}" rpy="${pi/2} 0 0" />
+        <origin xyz="-0.01 ${-wheel_offset_y} ${wheel_radius}" rpy="${pi/2} 0 0" />
         <axis xyz="0 0 -1"/>
     </joint>
